File: Hardware/WeatherStation-MM-Carrier.brd (EAGLE design)
At the start: 64.8 x 58.4 mm, 148 parts, among them J11 microSD, J13 RJ11 - WIND, J2 JTAG, J3 QWIIC_RIGHT_ANGLE, J7 RJ11 - RAIN, J9 MICROMOD-2222-C, U1 BME280, U2 VEML6075, U3 AS3935, U5 AP7361C-33FGE

Commit message: Routing
Parts:
- moved U$34 51.2 mm to (71.1, 40.6)
- moved U$62 50.1 mm to (67.4, 40.9)
- moved C5 49.9 mm to (71.1, 45.7)
- moved U2 49.9 mm to (71.1, 43.2)
- moved C3 49.3 mm to (71.1, 55.9)
- moved C4 49.3 mm to (71.1, 54.6)
- moved R7 49.3 mm to (71.1, 53.3)
- moved U1 49.3 mm to (74.9, 54.6)
- moved R21 49.3 mm to (78.7, 54.6)
- moved U$20 48.1 mm to (69.8, 50.8)
- moved U$11 45.2 mm to (50.3, 57.1)
- moved U$54 45.2 mm to (50.3, 57.1)
- moved C8 30.5 mm to (14.0, 52.1), turned to 180 degrees
- moved L1 30.5 mm to (14.0, 55.9), turned to 180 degrees
- moved R6 30.5 mm to (14.0, 53.3), turned to 0 degrees
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Routing:
- net 3.3V: track 0.00 -> 138.6 mm, vias 0 -> 3
- net VIN: track 0.00 -> 70.7 mm, vias 0 -> 3
- net PWM1: track 0.00 -> 55.6 mm, vias 0 -> 2
- net SD_CLK: track 0.00 -> 54.7 mm, vias 0 -> 2
- net SD_DAT0: track 0.00 -> 51.9 mm, vias 0 -> 2
- net SD_DAT1: track 0.00 -> 49.7 mm, vias 0 -> 2
- net SPI_CLK: track 0.00 -> 45.7 mm, vias 0 -> 4
- net SPI_MOSI: track 0.00 -> 44.4 mm, vias 0 -> 3
- net I2C_SDA: track 0.00 -> 44.4 mm, vias 0 -> 3
- net I2C_SCL: track 0.00 -> 42.9 mm, vias 0 -> 1
- net SPI_MISO: track 0.00 -> 42.4 mm, vias 0 -> 3
- net SPI_!CS!: track 0.00 -> 42.3 mm, vias 0 -> 4
- net SD_CMD: track 0.00 -> 39.2 mm, vias 0 -> 2
- net RTC_3V: track 0.00 -> 31.7 mm
- net SD_DAT2: track 0.00 -> 31.6 mm, vias 0 -> 2
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
Commit message: Routing
Parts:
- moved C3 43.2 mm to (33.0, 35.6)
- moved C4 43.2 mm to (33.0, 34.3)
- moved R7 43.2 mm to (33.0, 33.0)
- moved U1 42.1 mm to (38.1, 34.3)
- moved R21 41.0 mm to (43.2, 34.3)
- moved U$20 41.0 mm to (34.3, 30.5)
- moved U$34 35.7 mm to (35.6, 43.2)
- moved U$62 34.5 mm to (33.0, 43.2)
- moved C5 34.4 mm to (36.8, 48.3)
- moved U2 34.4 mm to (36.8, 45.7)
- moved U$55 0.51 mm to (27.0, 32.4)
Routing:
- net 3.3V: track 138.6 -> 154.2 mm
Other:
- outline, holes or cut-outs redrawn
