File: Hardware/WeatherStation-MM-Carrier.sch (EAGLE design)
At the start: 87 parts, among them J11 microSD, J13 RJ11 - WIND, J15 MICROMOD-2222-C, J2 JTAG, J3 QWIIC_RIGHT_ANGLE, J7 RJ11 - RAIN, U1 BME280, U2 VEML6075, U3 AS3935, U5 AP7361C-33FGEUDFN-8

Commit message: Added pullup resistor on CS line for SD card
Parts:
- added R12: 100k, SparkFun-Resistors:100KOHM-0603-1/10W-1%
Connections:
- net 3.3V: now also R12.2
- net SD_!CS!: now also R12.1
Changed lines of the file:
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@@
 <?xml version="1.0" encoding="utf-8"?>
 <!DOCTYPE eagle SYSTEM "eagle.dtd">
-<eagle version="9.4.2">
+<eagle version="9.5.2">
 <drawing>
 <settings>
-<setting alwaysvectorfont="yes"/>
+<setting alwaysvectorfont="no"/>
 <setting verticaltext="up"/>
 </settings>
@@
 <part name="JP6" library="SparkFun-Jumpers" deviceset="JUMPER-SMT_2_NO" device="_SILK" package3d_urn="urn:adsk.eagle:package:39279/1" value="VE"/>
 <part name="TP1" library="SparkFun-Connectors" deviceset="TEST-POINT" device="3X5"/>
+<part name="R12" library="SparkFun-Resistors" deviceset="100KOHM" device="-0603-1/10W-1%" value="100k"/>
+<part name="SUPPLY15" library="SparkFun-PowerSymbols" deviceset="3.3V" device=""/>
 </parts>
 <sheets>
@@
 <attribute name="VALUE" x="256.54" y="15.24" size="1.778" layer="96" font="vector"/>
 </instance>
+<instance part="R12" gate="G$1" x="154.94" y="147.32" smashed="yes" rot="R90">
+<attribute name="NAME" x="153.416" y="147.32" size="1.778" layer="95" font="vector" rot="R90" align="bottom-center"/>
+<attribute name="VALUE" x="156.464" y="147.32" size="1.778" layer="96" font="vector" rot="R90" align="top-center"/>
+</instance>
+<instance part="SUPPLY15" gate="G$1" x="154.94" y="154.94" smashed="yes">
+<attribute name="VALUE" x="154.94" y="157.734" size="1.778" layer="96" align="bottom-center"/>
+</instance>
 </instances>
 <busses>
@@
 <pinref part="SUPPLY14" gate="G$1" pin="3.3V"/>
 <wire x1="381" y1="261.62" x2="381" y2="264.16" width="0.1524" layer="91"/>
+</segment>
+<segment>
+<pinref part="R12" gate="G$1" pin="2"/>
+<pinref part="SUPPLY15" gate="G$1" pin="3.3V"/>
+<wire x1="154.94" y1="154.94" x2="154.94" y2="152.4" width="0.1524" layer="91"/>
 </segment>
 </net>
@@
 </segment>
 <segment>
-<wire x1="134.62" y1="139.7" x2="137.16" y2="139.7" width="0.1524" layer="91"/>
-<label x="137.16" y="139.7" size="1.27" layer="95" xref="yes"/>
+<wire x1="134.62" y1="139.7" x2="154.94" y2="139.7" width="0.1524" layer="91"/>
+<label x="157.48" y="139.7" size="1.27" layer="95" xref="yes"/>
 <pinref part="J15" gate="J1" pin="SPI_!CS!/SDIO_DATA3"/>
-</segment>
-</net>
+<pinref part="R12" gate="G$1" pin="1"/>
+<wire x1="154.94" y1="139.7" x2="157.48" y2="139.7" width="0.1524" layer="91"/>
+<wire x1="154.94" y1="139.7" x2="154.94" y2="142.24" width="0.1524" layer="91"/>
+<junction x="154.94" y="139.7"/>
+</segment>
+</net>

Commit message: Changed lightning CS from 10k to 100k (for ESP bootloading)
Parts:
- R19: value 10k -> 100k; device SparkFun-Resistors:10KOHM-0603-1/10W-1% -> SparkFun-Resistors:100KOHM-0603-1/10W-1%
Other:
- note removed: "~20 minute charge time"
Changed lines of the file:
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@@
 <?xml version="1.0" encoding="utf-8"?>
 <!DOCTYPE eagle SYSTEM "eagle.dtd">
-<eagle version="9.5.2">
+<eagle version="9.4.2">
 <drawing>
 <settings>
-<setting alwaysvectorfont="no"/>
+<setting alwaysvectorfont="yes"/>
 <setting verticaltext="up"/>
 </settings>
@@
 <part name="C8" library="SparkFun-Capacitors" deviceset="1.0NF/1000PF" device="-0603-50V-10%" value="1nF"/>
 <part name="R6" library="SparkFun-Resistors" deviceset="10KOHM" device="-0603-1/10W-1%" value="10k"/>
-<part name="R19" library="SparkFun-Resistors" deviceset="10KOHM" device="-0603-1/10W-1%" value="10k"/>
+<part name="R19" library="SparkFun-Resistors" deviceset="100KOHM" device="-0603-1/10W-1%" value="100k"/>
 <part name="SUPPLY29" library="SparkFun-PowerSymbols" deviceset="3.3V" device=""/>
 <part name="L1" library="SparkFun-Coils" deviceset="MA5532-AE" device="" value="100uH"/>
@@
 <text x="35.56" y="200.66" size="1.778" layer="97" font="vector" rot="R90">0.65uA Leakage
 0.3V drop at 10mA</text>
-<text x="48.26" y="180.34" size="1.778" layer="97" font="vector">~20 minute charge time</text>
 <text x="48.26" y="182.88" size="1.778" layer="97" font="vector">1mAhr Capacity</text>
 <text x="71.12" y="210.82" size="1.778" layer="97" font="vector">This is the penny-in-the-fuse jumper.

Commit message: Updated M.2 connector with increased tCream layer. Regenerated production files
Connections:
- net SPI_CIPO: now also J15.SPI_SDI/SDIO_DATA0; no longer J15.SPI_MISO/SDIO_DATA0
- net SPI_COPI: now also J15.SPI_SDO/SDIO_CMD; no longer J15.SPI_MOSI/SDIO_CMD
Changed lines of the file:
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@@
 <wire x1="134.62" y1="149.86" x2="137.16" y2="149.86" width="0.1524" layer="91"/>
 <label x="137.16" y="149.86" size="1.27" layer="95" xref="yes"/>
-<pinref part="J15" gate="J1" pin="SPI_MOSI/SDIO_CMD"/>
+<pinref part="J15" gate="J1" pin="SPI_SDO/SDIO_CMD"/>
 </segment>
 </net>
@@
 <wire x1="134.62" y1="147.32" x2="137.16" y2="147.32" width="0.1524" layer="91"/>
 <label x="137.16" y="147.32" size="1.27" layer="95" xref="yes"/>
-<pinref part="J15" gate="J1" pin="SPI_MISO/SDIO_DATA0"/>
+<pinref part="J15" gate="J1" pin="SPI_SDI/SDIO_DATA0"/>
 </segment>
 </net>
