File: Hardware/Weather-MM-Carrier.brd (EAGLE design)
At the start: 67.3 x 58.4 mm, 157 parts, among them J11 microSD, J13 RJ11 - WIND, J15 MICROMOD-2222-C, J2 JTAG, J3 QWIIC_RIGHT_ANGLE, J7 RJ11 - RAIN, U1 BME280, U2 VEML6075, U3 AS3935, U5 AP7361C-33FGEUDFN-8

Commit message: Implemented SPI bus changes
Re-panelized and new gerbers
Connections:
- net SD_!CS!: now also J15.55; no longer J15.70
- net SPI_CIPO: now also J15.61; no longer J15.64
- net SPI_COPI: now also J15.59; no longer J15.62
- net SPI_SCK: now also J15.57; no longer J15.60
Routing:
- net SPI_SCK: track 74.5 -> 78.6 mm
- net SPI_CIPO: track 71.8 -> 74.7 mm
- net SPI_COPI: track 80.2 -> 82.1 mm
- net PWM0: track 40.8 -> 42.0 mm
- net PWM1: track 35.0 -> 34.2 mm
- net HEADER_!CS!: track 48.3 -> 49.1 mm
Other:
- board text added: "v11"
- board text removed: "v10"
