File: Hardware/Weather-MM-Carrier.sch (EAGLE design)
At the start: 88 parts, among them J11 microSD, J13 RJ11 - WIND, J15 MICROMOD-2222-C, J2 JTAG, J3 QWIIC_RIGHT_ANGLE, J7 RJ11 - RAIN, U1 BME280, U2 VEML6075, U3 AS3935, U5 AP7361C-33FGEUDFN-8

Commit message: Implemented SPI bus changes
Re-panelized and new gerbers
Connections:
- net SD_!CS!: now also J15.SPI_!CS!; no longer J15.SPI_!CS!/SDIO_DATA3
- net SPI_CIPO: now also J15.SPI_SDI; no longer J15.SPI_SDI/SDIO_DATA0
- net SPI_COPI: now also J15.SPI_SDO; no longer J15.SPI_SDO/SDIO_CMD
- net SPI_SCK: now also J15.SPI_SCK; no longer J15.SPI_SCK/SDIO_CLK
Other:
- note added: "v11"
- note removed: "v10"
- moved on the sheet: R12
Changed lines of the file:
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@@
 <text x="391.16" y="226.06" size="1.778" layer="97" font="vector" align="center">I2C address: 0x10</text>
 <text x="386.08" y="200.66" size="1.778" layer="97" font="vector" align="center">Select SPI mode</text>
-<text x="419.1" y="7.62" size="2.54" layer="94" font="vector">v10</text>
+<text x="419.1" y="7.62" size="2.54" layer="94" font="vector">v11</text>
 <text x="388.62" y="259.08" size="1.778" layer="97" font="vector">Cut this jumper if you want to
 remove from power add an
@@
 <attribute name="VALUE" x="256.54" y="15.24" size="1.778" layer="96" font="vector"/>
 </instance>
-<instance part="R12" gate="G$1" x="154.94" y="147.32" smashed="yes" rot="R90">
-<attribute name="NAME" x="153.416" y="147.32" size="1.778" layer="95" font="vector" rot="R90" align="bottom-center"/>
-<attribute name="VALUE" x="156.464" y="147.32" size="1.778" layer="96" font="vector" rot="R90" align="top-center"/>
-</instance>
-<instance part="SUPPLY15" gate="G$1" x="154.94" y="154.94" smashed="yes">
-<attribute name="VALUE" x="154.94" y="157.734" size="1.778" layer="96" align="bottom-center"/>
+<instance part="R12" gate="G$1" x="154.94" y="134.62" smashed="yes" rot="R90">
+<attribute name="NAME" x="153.416" y="134.62" size="1.778" layer="95" font="vector" rot="R90" align="bottom-center"/>
+<attribute name="VALUE" x="156.464" y="134.62" size="1.778" layer="96" font="vector" rot="R90" align="top-center"/>
+</instance>
+<instance part="SUPPLY15" gate="G$1" x="154.94" y="142.24" smashed="yes">
+<attribute name="VALUE" x="154.94" y="145.034" size="1.778" layer="96" align="bottom-center"/>
 </instance>
 </instances>
@@
 </segment>
 <segment>
-<wire x1="134.62" y1="152.4" x2="137.16" y2="152.4" width="0.1524" layer="91"/>
-<label x="137.16" y="152.4" size="1.27" layer="95" xref="yes"/>
-<pinref part="J15" gate="J1" pin="SPI_SCK/SDIO_CLK"/>
-</segment>
-<segment>
 <pinref part="J5" gate="G$1" pin="1"/>
 <wire x1="223.52" y1="83.82" x2="220.98" y2="83.82" width="0.1524" layer="91"/>
@@
 <wire x1="391.16" y1="187.96" x2="396.24" y2="187.96" width="0.1524" layer="91"/>
 <label x="396.24" y="187.96" size="1.27" layer="95" xref="yes"/>
+</segment>
+<segment>
+<pinref part="J15" gate="J1" pin="SPI_SCK"/>
+<wire x1="134.62" y1="134.62" x2="137.16" y2="134.62" width="0.1524" layer="91"/>
+<label x="137.16" y="134.62" size="1.27" layer="95" xref="yes"/>
 </segment>
 </net>
@@
 <pinref part="R12" gate="G$1" pin="2"/>
 <pinref part="SUPPLY15" gate="G$1" pin="3.3V"/>
-<wire x1="154.94" y1="154.94" x2="154.94" y2="152.4" width="0.1524" layer="91"/>
+<wire x1="154.94" y1="142.24" x2="154.94" y2="139.7" width="0.1524" layer="91"/>
 </segment>
 </net>
@@
 </segment>
 <segment>
-<wire x1="134.62" y1="149.86" x2="137.16" y2="149.86" width="0.1524" layer="91"/>
-<label x="137.16" y="149.86" size="1.27" layer="95" xref="yes"/>
-<pinref part="J15" gate="J1" pin="SPI_SDO/SDIO_CMD"/>
+<pinref part="J15" gate="J1" pin="SPI_SDO"/>
+<wire x1="134.62" y1="132.08" x2="137.16" y2="132.08" width="0.1524" layer="91"/>
+<label x="137.16" y="132.08" size="1.27" layer="95" xref="yes"/>
 </segment>
 </net>
@@
 </segment>
 <segment>
-<wire x1="134.62" y1="147.32" x2="137.16" y2="147.32" width="0.1524" layer="91"/>
-<label x="137.16" y="147.32" size="1.27" layer="95" xref="yes"/>
-<pinref part="J15" gate="J1" pin="SPI_SDI/SDIO_DATA0"/>
+<pinref part="J15" gate="J1" pin="SPI_SDI"/>
+<wire x1="134.62" y1="129.54" x2="137.16" y2="129.54" width="0.1524" layer="91"/>
+<label x="137.16" y="129.54" size="1.27" layer="95" xref="yes"/>
 </segment>
 </net>
@@
 </segment>
 <segment>
-<wire x1="134.62" y1="139.7" x2="154.94" y2="139.7" width="0.1524" layer="91"/>
-<label x="157.48" y="139.7" size="1.27" layer="95" xref="yes"/>
-<pinref part="J15" gate="J1" pin="SPI_!CS!/SDIO_DATA3"/>
+<pinref part="J15" gate="J1" pin="SPI_!CS!"/>
+<wire x1="134.62" y1="127" x2="154.94" y2="127" width="0.1524" layer="91"/>
+<label x="157.48" y="127" size="1.27" layer="95" xref="yes"/>
 <pinref part="R12" gate="G$1" pin="1"/>
-<wire x1="154.94" y1="139.7" x2="157.48" y2="139.7" width="0.1524" layer="91"/>
-<wire x1="154.94" y1="139.7" x2="154.94" y2="142.24" width="0.1524" layer="91"/>
-<junction x="154.94" y="139.7"/>
-</segment>
-</net>
+<wire x1="154.94" y1="127" x2="157.48" y2="127" width="0.1524" layer="91"/>
+<wire x1="154.94" y1="127" x2="154.94" y2="129.54" width="0.1524" layer="91"/>
+<junction x="154.94" y="127"/>
+</segment>
+</net>
